Commit message: package name update

File: src/safety_shield_node/urdf/ur_robots/ur3.urdf (robot description, URDF)
Before this commit: robot ur3, 13 links, 12 joints
Links:
- link base_link_inertia: geometry collision mesh filename=package://safety_shield_node/urdf/ur_robots/meshes/ur3/coll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; visual mesh filename=package://safety_shield_node/urdf/ur_robots/meshes/ur3/visu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
- link forearm_link: geometry collision mesh filename=package://safety_shield_node/urdf/ur_robots/meshes/ur3/coll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; visual mesh filename=package://safety_shield_node/urdf/ur_robots/meshes/ur3/visu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
- link shoulder_link: geometry collision mesh filename=package://safety_shield_node/urdf/ur_robots/meshes/ur3/coll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; visual mesh filename=package://safety_shield_node/urdf/ur_robots/meshes/ur3/visu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
- link upper_arm_link: geometry collision mesh filename=package://safety_shield_node/urdf/ur_robots/meshes/ur3/coll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; visual mesh filename=package://safety_shield_node/urdf/ur_robots/meshes/ur3/visu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
- link wrist_1_link: geometry collision mesh filename=package://safety_shield_node/urdf/ur_robots/meshes/ur3/coll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; visual mesh filename=package://safety_shield_node/urdf/ur_robots/meshes/ur3/visu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
- link wrist_2_link: geometry collision mesh filename=package://safety_shield_node/urdf/ur_robots/meshes/ur3/coll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; visual mesh filename=package://safety_shield_node/urdf/ur_robots/meshes/ur3/visu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
- link wrist_3_link: geometry collision mesh filename=package://safety_shield_node/urdf/ur_robots/meshes/ur3/coll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; visual mesh filename=package://safety_shield_node/urdf/ur_robots/meshes/ur3/visu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
