Commit message: initi working version multiple waypoints

File: src/safety_shield_node/urdf/panda/panda.urdf (robot description, URDF)
Before this commit: robot panda, 13 links, 12 joints
Links:
- added link world
Joints:
- added joint world_to_base: type fixed, parent world, child panda_link0, origin xyz=0 0 0 rpy=0 0 0
